Commit message: tuning side arm URDF

File: src/side_arm_control/urdf/side_arm.urdf (robot description, URDF)
Before this commit: robot side_arm, 10 links, 9 joints
Links:
- removed link side_arm_base
- added link side_arm_origin; visual sphere radius=0.01
Joints:
- joint base_to_x_rail: parent side_arm_base -> side_arm_origin

Commit message: urdf and camera tf edit

File: src/side_arm_control/urdf/side_arm.urdf (robot description, URDF)
Before this commit: robot side_arm, 10 links, 9 joints
Joints:
- joint joint_x: axis 1 0 0 -> -1 0 0

Commit message: grid alignment

File: src/side_arm_control/urdf/side_arm.urdf (robot description, URDF)
Before this commit: robot side_arm, 10 links, 9 joints
Joints:
- joint servo_to_hook: origin xyz=-0.01 0.009 0.07 rpy=0 0 0 -> xyz=0.01 -0.009 0.07 rpy=0 0 0

Commit message: urdf update

File: src/side_arm_control/urdf/side_arm.urdf (robot description, URDF)
Before this commit: robot side_arm, 10 links, 9 joints
Joints:
- joint servo_to_hook: origin xyz=0.01 -0.009 0.07 rpy=0 0 0 -> xyz=0.01 0.009 0.07 rpy=0 0 0

Commit message: attach camera in rviz

File: src/side_arm_control/urdf/side_arm.urdf (robot description, URDF)
Before this commit: robot side_arm, 10 links, 9 joints
Joints:
- joint joint_servo: axis 0 1 0 -> 0 0 1

Commit message: hybrid hw and sw visualization, camera angle

File: src/side_arm_control/urdf/side_arm.urdf (robot description, URDF)
Before this commit: robot side_arm, 10 links, 9 joints
Joints:
- joint hook_to_camera: origin xyz=0 0 0.05 rpy=0 3.1416 0 -> xyz=0 0 0.05 rpy=0 0 0

Commit message: adjust camera joint

File: src/side_arm_control/urdf/side_arm.urdf (robot description, URDF)
Before this commit: robot side_arm, 10 links, 9 joints
Joints:
- removed joint hook_to_camera
- added joint y_carriage_to_camera: type fixed, parent y_carriage_link, child camera_link, origin xyz=0 0 0.05 rpy=0 3.1416 0

Commit message: reconcile double camera frame

File: src/side_arm_control/urdf/side_arm.urdf (robot description, URDF)
Before this commit: robot side_arm, 10 links, 9 joints
Links:
- removed link camera_link
- added link camera_frame; visual box size=0.02 0.015 0.015
Joints:
- joint y_carriage_to_camera: child camera_link -> camera_frame; origin xyz=0 0 0.05 rpy=0 3.1416 0 -> xyz=0 -0.05 0 rpy=1.5708 0 0

Commit message: camera grid published correctly

File: src/side_arm_control/urdf/side_arm.urdf (robot description, URDF)
Before this commit: robot side_arm, 10 links, 9 joints
Joints:
- joint y_carriage_to_camera: origin xyz=0 -0.05 0 rpy=1.5708 0 0 -> xyz=0 -0.05 0 rpy=0 3.1416 0

Commit message: tune camera placement and check tf frames

File: src/side_arm_control/urdf/side_arm.urdf (robot description, URDF)
Before this commit: robot side_arm, 10 links, 9 joints
Joints:
- joint y_carriage_to_camera: origin xyz=0 -0.05 0 rpy=0 3.1416 0 -> xyz=0.01 0.03 0.03 rpy=0 3.1416 0

Commit message: update camera attributes

File: src/side_arm_control/urdf/side_arm.urdf (robot description, URDF)
Before this commit: robot side_arm, 10 links, 9 joints
Joints:
- joint y_carriage_to_camera: origin xyz=0.01 0.03 0.03 rpy=0 3.1416 0 -> xyz=0.01 0.03 0.1 rpy=0 3.0 0

Commit message: calibrated URDF with camera view in correct place

File: src/side_arm_control/urdf/side_arm.urdf (robot description, URDF)
Before this commit: robot side_arm, 10 links, 9 joints
Links:
- link y_carriage_link: geometry visual box size=0.03 0.04 0.07
- link y_rail_link: geometry visual box size=0.004 0.05 0.02
- link z_rail_link: geometry visual box size=0.02 0.004 0.20
Joints:
- joint joint_servo: origin xyz=0 0 0.02 rpy=0 0 0 -> xyz=0 0.02 0.02 rpy=0 0 0
- joint joint_y: limit lower=0.0 upper=0.2 effort=10 velocity=0.05 -> lower=0.0 upper=0.1 effort=10 velocity=0.05
- joint joint_z: limit lower=0.0 upper=0.15 effort=10 velocity=0.01 -> lower=0.0 upper=0.20 effort=10 velocity=0.01
- joint servo_to_hook: origin xyz=0.01 0.009 0.07 rpy=0 0 0 -> xyz=0.01 0.009 -0.18 rpy=0 0 0
- joint x_carriage_to_y_rail: origin xyz=0 0 0 rpy=0 0 0 -> xyz=0 0.095 0 rpy=0 0 0
- joint y_carriage_to_camera: origin xyz=0.01 0.03 0.1 rpy=0 3.0 0 -> xyz=0.04 0.08 -0.05 rpy=0.1 3.2116 3.1416
- joint y_carriage_to_z_rail: origin xyz=0 0 0 rpy=0 0 0 -> xyz=0 0.07 0 rpy=0.1 0 0
